Commit message: Atlas visualization in color

File: atlas_description/urdf/atlas.urdf (robot description, URDF)
Before this commit: robot Atlas, 4 links, 3 joints
Links:
- removed link base_link
- removed link lwheel_link
- removed link rwheel_link
- added link base, mass 0.499281541152724; collision mesh filename=package://atlas_description/meshes/base_link.obj; visual mesh filename=package://atlas_description/meshes/base_link.obj
- added link lwheel, mass 0.166945648009266; collision mesh filename=package://atlas_description/meshes/wheel.obj; visual mesh filename=package://atlas_description/meshes/wheel.obj
- added link rwheel, mass 0.166945648008949; collision mesh filename=package://atlas_description/meshes/wheel.obj; visual mesh filename=package://atlas_description/meshes/wheel.obj
Joints:
- joint dummy_joint: child base_link -> base
- joint lwheel_joint: child lwheel_link -> lwheel; origin xyz=-0.0459 0.0476 -0.013 rpy=1.5708 0 -1.5708 -> xyz=0.0459 0.0776 -0.013 rpy=1.5708 0 -3.1415; parent base_link -> base
- joint rwheel_joint: child rwheel_link -> rwheel; origin xyz=0.0459 0.0476 -0.013 rpy=1.5708 0 1.5708 -> xyz=0.0459 -0.0776 -0.013 rpy=1.5708 0 0; parent base_link -> base

File: atlas_description/urdf/atlasfixed.urdf (robot description, URDF)
Before this commit: robot Atlas, 3 links, 2 joints
Links:
- link base: geometry collision mesh filename=package://atlas_description/meshes/base_link.obj; visual mesh filename=package://atlas_description/meshes/base_link.obj
- link lwheel: geometry collision mesh filename=package://atlas_description/meshes/wheel.obj; visual mesh filename=package://atlas_description/meshes/wheel.obj
- link rwheel: geometry collision mesh filename=package://atlas_description/meshes/wheel.obj; visual mesh filename=package://atlas_description/meshes/wheel.obj
Joints:
- joint lwheel_joint: origin xyz=0.0459 0.0476 -0.013 rpy=1.5708 0 -3.1415 -> xyz=0.0459 0.0776 -0.013 rpy=1.5708 0 -3.1415
- joint rwheel_joint: origin xyz=0.0459 -0.0476 -0.013 rpy=1.5708 0 0 -> xyz=0.0459 -0.0776 -0.013 rpy=1.5708 0 0
